File: pcb/V001/V001.kicad_pcb (KiCad board)
At the start: 2 copper layers, 76 x 88 mm, 128 parts, among them J1 USB_B_Micro, J10 CAN, J2 Display, J3 WHBUS, J4 CU, J5 CD, J6 Conn_01x04, J7 8P8C_LED_Shielded, J8 Conn_01x08, Q1 Q_NPN_BEC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

Commit message: merged repository
Routing:
- net GND: vias 66 -> 65
- net +5V: vias 2 -> 3
Other:
- board text added: "55mm hoch"
- board text added: "70mm hoch"
- board text added: "Wandstärke 1,5mm + 0,5mm an manchen Stellen für Clipse"
Changed lines of the file:
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@@
   (general
     (thickness 1.6)
-    (drawings 22)
+    (drawings 40)
     (tracks 1461)
     (zones 0)
@@
     (38 B.Mask user hide)
     (39 F.Mask user hide)
-    (40 Dwgs.User user hide)
+    (40 Dwgs.User user)
     (41 Cmts.User user hide)
     (42 Eco1.User user hide)
@@
     )
   )
+  (gr_text "70mm hoch" (at 74 123.5) (layer Dwgs.User)
+    (effects (font (size 1 1) (thickness 0.15)))
+  )
+  (gr_text "55mm hoch" (at 89 123.5) (layer Dwgs.User)
+    (effects (font (size 1 1) (thickness 0.15)))
+  )
+  (gr_line (start 89 77.5) (end 89 122.5) (layer Dwgs.User) (width 0.15))
+  (gr_text "Wandstärke 1,5mm + 0,5mm an \nmanchen Stellen für Clipse" (at 159.5 87.5) (layer Dwgs.User)
+    (effects (font (size 1 1) (thickness 0.15)))
+  )
+  (gr_line (start 144 117.5) (end 144 100) (layer Dwgs.User) (width 0.15))
+  (gr_line (start 150 117.5) (end 144 117.5) (layer Dwgs.User) (width 0.15))
+  (gr_line (start 150 120) (end 150 117.5) (layer Dwgs.User) (width 0.15))
+  (gr_line (start 150 145) (end 150 120) (layer Dwgs.User) (width 0.15))
+  (gr_line (start 100 145) (end 150 145) (layer Dwgs.User) (width 0.15))
+  (gr_line (start 100 122.5) (end 100 145) (layer Dwgs.User) (width 0.15))
+  (gr_line (start 74 122.5) (end 100 122.5) (layer Dwgs.User) (width 0.15))
+  (gr_line (start 74 77.5) (end 74 122.5) (layer Dwgs.User) (width 0.15))
+  (gr_line (start 100 77.5) (end 74 77.5) (layer Dwgs.User) (width 0.15))
+  (gr_line (start 100 55) (end 100 77.5) (layer Dwgs.User) (width 0.15))
+  (gr_line (start 150 55) (end 100 55) (layer Dwgs.User) (width 0.15))
+  (gr_line (start 150 82.5) (end 150 55) (layer Dwgs.User) (width 0.15))
+  (gr_line (start 144 82.5) (end 150 82.5) (layer Dwgs.User) (width 0.15))
+  (gr_line (start 144 100) (end 144 82.5) (layer Dwgs.User) (width 0.15))
   (gr_line (start 150 144) (end 150 120) (layer Edge.Cuts) (width 0.15))
   (gr_line (start 150 80) (end 150 56) (layer Edge.Cuts) (width 0.15))
@@
   (via (at 109.855 115.697) (size 0.7) (drill 0.3) (layers F.Cu B.Cu) (net 2))
   (via (at 110.998 115.697) (size 0.7) (drill 0.3) (layers F.Cu B.Cu) (net 2))
-  (via (at 112.141 115.697) (size 0.7) (drill 0.3) (layers F.Cu B.Cu) (net 2))
+  (via (at 112.141 115.697) (size 0.7) (drill 0.3) (layers F.Cu B.Cu) (net 44))
   (via (at 113.284 115.697) (size 0.7) (drill 0.3) (layers F.Cu B.Cu) (net 2))
   (via (at 102.997 125.476) (size 0.7) (drill 0.3) (layers F.Cu B.Cu) (net 2))
